Commit message: Replace CuRobo with PyRoki

File: assets/ur3e_custom.urdf (robot description, URDF)
Before this commit: robot ur, 13 links, 12 joints
Joints:
- joint wrist_3_joint: limit effort=9.0 velocity=6.283185307179586 -> lower=-12.56637 upper=12.56637 effort=9.0 velocity=6.283185307179586; type continuous -> revolute

Commit message: Add camera mount

File: assets/ur3e_custom.urdf (robot description, URDF)
Before this commit: robot ur, 13 links, 12 joints
Links:
- added link camera_color_optical_frame
- added link camera_mount_link, mass 0.05; collision mesh filename=package://ur_description/robot_camera_mount_1.stl; visual mesh filename=package://ur_description/robot_camera_mount_1.stl
- added link d455_link, mass 0.072; collision mesh filename=package://ur_description/d455.stl; visual mesh filename=package://ur_description/d455.stl
Joints:
- added joint camera_mount-d455: type fixed, parent camera_mount_link, child d455_link, origin xyz=0 0.06573 0.006 rpy=0 0 0
- added joint d455-camera_color_optical: type fixed, parent d455_link, child camera_color_optical_frame, origin xyz=0.0325 0 0.026 rpy=-1.5707963267948966 0 -1.5707963267948966
- added joint tool0-camera_mount: type fixed, parent tool0, child camera_mount_link, origin xyz=0 0 0 rpy=0 0 0

Commit message: Stable: Complete correct 3-axis grip rotation mapping and joint limit protection

File: assets/ur3e_custom.urdf (robot description, URDF)
Before this commit: robot ur, 16 links, 15 joints
Links:
- added link wrist_1_motor_link; collision cylinder length=0.065 radius=0.033
- added link wrist_2_motor_link; collision sphere radius=0.031
- link camera_mount_link: geometry collision box size=0.116 0.128 0.016; collision sphere radius=0.010
- link d455_link: geometry collision cylinder length=0.138 radius=0.028; visual mesh filename=package://ur_description/d455.stl
- link forearm_link: geometry collision cylinder length=0.170 radius=0.030; visual mesh filename=package://ur_description/meshes/ur3e/visual/forearm.dae
- link shoulder_link: geometry collision cylinder length=0.070 radius=0.050; visual mesh filename=package://ur_description/meshes/ur3e/visual/shoulder.dae
- link upper_arm_link: geometry collision cylinder length=0.23355 radius=0.035; visual mesh filename=package://ur_description/meshes/ur3e/visual/upperarm.dae
- link wrist_1_link: geometry collision cylinder length=0.070 radius=0.030; visual mesh filename=package://ur_description/meshes/ur3e/visual/wrist1.dae
- link wrist_2_link: geometry collision cylinder length=0.070 radius=0.030; visual mesh filename=package://ur_description/meshes/ur3e/visual/wrist2.dae
- link wrist_3_link: geometry collision cylinder length=0.030 radius=0.0365; visual mesh filename=package://ur_description/meshes/ur3e/visual/wrist3.dae
Joints:
- added joint forearm-wrist_1_motor: type fixed, parent forearm_link, child wrist_1_motor_link, origin xyz=-0.2132 0 0.13105 rpy=0 0 0
- added joint wrist_1-wrist_2_motor: type fixed, parent wrist_1_link, child wrist_2_motor_link, origin xyz=0 -0.08535 0 rpy=1.570796327 0 0
- joint tool0-camera_mount: origin xyz=0 0 0 rpy=0 0 0 -> xyz=0 0 0 rpy=0 0 -1.5707963267948966
